File: module/Main Module/搭載型点火装置回路図draft.kicad_sch (KiCad schematic)
At the start: 27 parts, among them Q1 NPN, Q2 BS250, Q3 BS170, SW1 SW_DPDT_x2

Commit message: NewChanges20231130
Parts:
- removed R13, R14, R8: R_US, symbol Device:R_US
- R7: value R_US -> 5+
Connections:
- net at FLIGHTPIN., IGNITER.: now also Q3.1 (D), SW1.3 (C); no longer SW1.1 (A)
- new net: FLIGHTPIN., IGNITER., SW1.1 (A)
- new net 3V3: RP1. (GND), TWE1. (VCC)
Other:
- note added: "GNDにつける必要ありますか？"
- note added: "ON→0.05mV, 0.01A"
- moved on the sheet: BZ1, D1, D2, D3, D4, FLIGHTPIN, IGNITER, INA1, Q1, Q2, Q3, R1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
