File: module/Main Module/BBM/BBM.kicad_sch (KiCad schematic)
At the start: 30 parts, among them Q1 NPN, Q2 BS250, Q3 BS170, SW1 SW_DPDT_x2, SW2 SW_Push

Commit message: KiCad & Program reviewed
Parts:
- removed R6: 10, symbol Device:R_US
- removed R8: R_US, symbol Device:R_US
- added R2: 5, symbol Device:R_US
- added R24, R25: R_US, symbol Device:R_US
- R1, R11, R12, R2: value R_US -> 100
- R13, R14: value R_US -> 10000
- R15: value 1 -> 10
- R3: value 30+ -> 100
- R4: value R_US -> 23
- R5: value 20 -> 1
- R7: value R_US -> 5
- R8: value R_US -> 1000
Connections:
- net Pow is gone; now on net TX: RP1. (GND)
- net BAT+: now also INA1. (Vs), R13.1, RP1. (GND), R24.1, R25.1
- net Earth: now also R2.1
- net SCL: now also R25.2
- net SDA: now also R24.2
- net TEST: now also RP1. (GND)
- net at D4.2 (A), R7.1: now also R2.2
- removed net POW: INA1. (Vs), R13.1
Other:
- note added: "0.05V 0.01A"
- note added: "0.1V"
- note added: "ON→0.3A"
- note added: "ON→30mA"
- note added: "ON→3V"
- note removed: "100mA"
- note removed: "3.5V"
- note removed: "SDA,SCLはプログラム中で PULLUPを指定"
- moved on the sheet: R7
