File: module/Main Module/BBM/_autosave-BBM.kicad_sch (KiCad schematic)
At the start: 30 parts, among them Q1 NPN, Q2 BS250, Q3 BS170, SW1 SW_DPDT_x2, SW2 SW_Push

Commit message: KiCad & Program reviewed
Parts:
- removed V1, V2: 1, symbol Simulation_SPICE:VDC
- added R2: 5, symbol Device:R_US
- added R24, R25: R_US, symbol Device:R_US
- R3: value 30 -> 100
- R4: value 100 -> 23
- R7: value 100 -> 5
Connections:
- net BAT+: now also R24.1, R25.1
- net Earth: now also R2.1
- net SCL: now also R25.2
- net SDA: now also R24.2
- net TEST: now also RP1. (GND)
- net at D4.2 (A), R7.1: now also R2.2
Other:
- note added: "0.05V 0.01A"
- note added: "0.1V"
- note added: "ON→0.3A"
- note added: "ON→30mA"
- note added: "ON→3V"
- note removed: "100mA 30Ω+"
- note removed: "SDA,SCLはプログラム中で PULLUPを指定"
- moved on the sheet: R7
